File: REF1198.kicad_sch (KiCad schematic)
At the start: 24 parts, among them J1 Bottom Edge Connector, J2 Top Edge Connector, J3 Smart_Card_Reader, SW1 SW_Push, U1 SST28LF040, U2 SST28LF040, U3 QuickLogic QL12X16B-XPL68C, U4 HDSP-7501, U5 74HC164

Commit message: Add files via upload
Parts:
- U1, U2: value SST28LF040 -> SST29LE010
Changed lines of the file:
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@@
 			)
 		)
-		(property "Value" "SST28LF040"
+		(property "Value" "SST29LE010"
 			(at 50.8 156.21 0)
 			(effects
@@
 			)
 		)
-		(property "Value" "SST28LF040"
+		(property "Value" "SST29LE010"
 			(at 52.07 29.21 0)
 			(effects
